File: ad4080_evb_experimenter.kicad_pcb (KiCad board)
At the start: 2 copper layers, 104.4 x 78.7 mm, 64 parts, among them J1 Conn_Coaxial, J2 Conn_Coaxial, J3 AudioJack2_Ground, J4 Conn_02x01, J5 Conn_02x01, J6 Conn_Coaxial, SW1 SW_Coded_SH-7050, U2 74LS163, U3 74HC04, X1 CXO_DIP8

Commit message: Add clock output SMA
Signed-off-by: Ioan Dragomir <ioan.dragomir@analog.com>
Parts:
- added J7: Conn_Coaxial, Connector_Coaxial:SMA_Amphenol_132289_EdgeMount, F.Cu at (73.9, 120.4)
- moved TP4 11.1 mm to (65.2, 118.7)
- moved JP10 2.92 mm to (53.2, 115.6)
Routing:
- net /CLK_1V8: track 8.89 -> 23.8 mm
- net Net-(JP10-B): track 32.9 -> 35.8 mm
- net Net-(JP10-A): track 14.8 -> 11.9 mm
- net GND: vias 82 -> 85
