File: ad4080_evb_experimenter.kicad_sch (KiCad schematic)
At the start: 63 parts, among them J1 Conn_Coaxial, J2 Conn_Coaxial, J3 AudioJack2_Ground, J4 Conn_02x01, J5 Conn_02x01, J6 Conn_Coaxial, SW1 SW_Coded_SH-7050, U2 74LS163, U3 74HC04, X1 CXO_DIP8

Commit message: Add clock output SMA
Signed-off-by: Ioan Dragomir <ioan.dragomir@analog.com>
Parts:
- added J7: Conn_Coaxial, Connector_Coaxial:SMA_Amphenol_132289_EdgeMount, symbol Connector:Conn_Coaxial
Connections:
- net CLK_1V8: now also J7.1 (In)
- net GND: now also J7.2 (Ext)
Changed lines of the file:
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@@
 	)
 	(junction
+		(at 152.4 168.91)
+		(diameter 0)
+		(color 0 0 0 0)
+	)
+	(junction
 		(at 149.86 46.99)
 		(diameter 0)
@@
 	(wire
 		(pts
+			(xy 152.4 168.91) (xy 154.94 168.91)
+		)
+		(stroke
+			(width 0)
+			(type default)
+		)
+	)
+	(wire
+		(pts
 			(xy 55.88 124.46) (xy 62.23 124.46)
 		)
@@
 	(wire
 		(pts
+			(xy 152.4 179.07) (xy 152.4 168.91)
+		)
+		(stroke
+			(width 0)
+			(type default)
+		)
+	)
+	(wire
+		(pts
 			(xy 256.54 139.7) (xy 256.54 132.08)
 		)
@@
 	(wire
 		(pts
-			(xy 143.51 168.91) (xy 154.94 168.91)
+			(xy 143.51 168.91) (xy 152.4 168.91)
 		)
 		(stroke
@@
 	(wire
 		(pts
+			(xy 154.94 179.07) (xy 152.4 179.07)
+		)
+		(stroke
+			(width 0)
+			(type default)
+		)
+	)
+	(wire
+		(pts
 			(xy 100.33 160.02) (xy 99.06 160.02)
 		)
@@
 	)
 	(symbol
+		(lib_id "Connector:Conn_Coaxial")
+		(at 160.02 179.07 0)
+		(unit 1)
+		(exclude_from_sim no)
+		(in_bom yes)
+		(on_board yes)
+		(dnp no)
+		(property "Reference" "J7"
+			(at 158.75 175.26 0)
+			(effects
+				(font
+					(size 1.27 1.27)
+				)
+				(justify left)
+			)
+		)
+		(property "Value" "Conn_Coaxial"
+			(at 157.734 175.514 0)
+			(effects
+				(font
+					(size 1.27 1.27)
+				)
+				(justify left)
+				(hide yes)
+			)
+		)
+		(property "Footprint" "Connector_Coaxial:SMA_Amphenol_132289_EdgeMount"
+			(at 160.02 179.07 0)
+			(effects
+				(font
+					(size 1.27 1.27)
+				)
+				(hide yes)
+			)
+		)
+		(property "Datasheet" " ~"
+			(at 160.02 179.07 0)
+			(effects
+				(font
+					(size 1.27 1.27)
+				)
+				(hide yes)
+			)
+		)
+		(property "Description" ""
+			(at 160.02 179.07 0)
+			(effects
+				(font
+					(size 1.27 1.27)
+				)
+				(hide yes)
+			)
+		)
+		(pin "1"
+		)
+		(pin "2"
+		)
+		(instances
+			(project "ad4080_evb_experimenter"
+				(path "/b69282a1-dfbe-4b32-8ce1-82537d42439c"
+					(reference "J7")
+					(unit 1)
+				)
+			)
+		)
+	)
+	(symbol
 		(lib_id "power:GND")
 		(at 199.39 144.78 0)
@@
 					(unit 1)
 				)
+			)
+		)
+	)
+	(symbol
+		(lib_id "power:GND")
+		(at 160.02 184.15 0)
+		(unit 1)
+		(exclude_from_sim no)
+		(in_bom yes)
+		(on_board yes)
+		(dnp no)
+		(fields_autoplaced yes)
+		(property "Reference" "#PWR012"
+			(at 160.02 190.5 0)
+			(effects
+				(font
+					(size 1.27 1.27)
+				)
+				(hide yes)
+			)
+		)
+		(property "Value" "GND"
+			(at 160.02 189.23 0)
+			(effects
+				(font
+					(size 1.27 1.27)
+				)
+			)
+		)
+		(property "Footprint" ""
+			(at 160.02 184.15 0)
+			(effects
+				(font
+					(size 1.27 1.27)
+				)
+				(hide yes)
+			)
+		)
+		(property "Datasheet" ""
+			(at 160.02 184.15 0)
+			(effects
+				(font
+					(size 1.27 1.27)
+				)
+				(hide yes)
+			)
+		)
+		(property "Description" ""
+			(at 160.02 184.15 0)
+			(effects
+				(font
+					(size 1.27 1.27)
+				)
+				(hide yes)
+			)
+		)
+		(pin "1"
+		)
+		(instances
+			(project "ad4080_evb_experimenter"
+				(path "/b69282a1-dfbe-4b32-8ce1-82537d42439c"
+					(reference "#PWR012")
+					(unit 1)
+				)
