File: minimal/ad4080_evb_experimenter_minimal.kicad_pcb (KiCad board)
At the start: 2 copper layers, 49 x 39.1 mm, 31 parts, among them J1 Conn_01x04_Pin, J2 AudioJack2_Ground, J3 Conn_01x04_Pin, J4 Conn_Coaxial, J5 Conn_Coaxial

Commit message: Adjust vias, routes, silkscreen
Signed-off-by: Ioan Dragomir <ioan.dragomir@analog.com>
Other:
- board text removed: "100"
- board text removed: "100uF"
- board text removed: "10K"
- board text removed: "10uF"
- board text removed: "1K"
- board text removed: "Attenuation"
- board text removed: "C1"
- board text removed: "C2"
- board text removed: "R1"
- board text removed: "R2"
